File: Diseño/Eagle/TeamRocket_PlacaSubsatélite/PlacaSubsatélite.brd (EAGLE design)
At the start: 55.9 x 50.5 mm, 8 parts, among them IC2 7806DT

Commit message: Update
Connections:
- removed net N$10: C2.1, IC2.2, U$2.VCC
- removed net N$12: C1.2, C2.2, U$3.GND, U$4.NA
- net DGND: now also C1.2, C2.2, IC2.3, U$3.GND, U$3.GND#2
- net N$1: now also U$4.NA; no longer JP1.2
- net N$2: now also JP1.2; no longer IC2.3
- net VCC: now also C2.1, IC2.2, U$2.VCC
Changed lines of the file:
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@@
 <contactref element="IC2" pad="1"/>
 <contactref element="U$3" pad="BAT"/>
-<contactref element="JP1" pad="2"/>
-<wire x1="62.23" y1="46.99" x2="62.49" y2="63.78" width="0" layer="19" extent="1-1"/>
-<wire x1="52.07" y1="41.78" x2="62.23" y2="46.99" width="0" layer="19" extent="1-1"/>
-<wire x1="48.26" y1="51.93" x2="52.07" y2="41.78" width="0" layer="19" extent="1-1"/>
+<contactref element="U$4" pad="NA"/>
+<wire x1="48.26" y1="51.93" x2="62.49" y2="63.78" width="0" layer="19" extent="1-1"/>
+<wire x1="52.07" y1="41.78" x2="48.26" y2="51.93" width="0" layer="19" extent="1-1"/>
+<wire x1="25.4" y1="29.21" x2="52.07" y2="41.78" width="0" layer="19" extent="1-1"/>
 </signal>
 <signal name="N$3">
@@
 <wire x1="38.1" y1="51.93" x2="59.42953125" y2="81.236640625" width="0" layer="19" extent="1-1"/>
 </signal>
-<signal name="N$12">
-<contactref element="C1" pad="2"/>
-<contactref element="U$4" pad="NA"/>
-<contactref element="U$3" pad="GND"/>
-<contactref element="C2" pad="2"/>
-<wire x1="52.07" y1="44.58" x2="48.26" y2="67.31" width="0" layer="19" extent="1-1"/>
-<wire x1="57.15" y1="44.58" x2="52.07" y2="44.58" width="0" layer="19" extent="1-1"/>
-<wire x1="25.4" y1="29.21" x2="52.07" y2="44.58" width="0" layer="19" extent="1-1"/>
-</signal>
-<signal name="N$10">
-<contactref element="IC2" pad="2"/>
-<contactref element="C2" pad="1"/>
-<contactref element="U$2" pad="VCC"/>
-<wire x1="67.05" y1="63.78" x2="57.15" y2="41.78" width="0" layer="19" extent="1-1"/>
-<wire x1="59.47294375" y1="72.98791875" x2="67.05" y2="63.78" width="0" layer="19" extent="1-1"/>
-</signal>
 <signal name="N$11">
 <contactref element="U$1" pad="SDO"/>
@@
 <contactref element="U$2" pad="GND"/>
 <contactref element="JP1" pad="1"/>
-<wire x1="63.5" y1="50.8" x2="59.429528125" y2="75.723040625" width="0" layer="19" extent="1-1"/>
-<wire x1="62.23" y1="44.45" x2="63.5" y2="50.8" width="0" layer="19" extent="1-1"/>
+<contactref element="C1" pad="2"/>
+<contactref element="C2" pad="2"/>
+<contactref element="IC2" pad="3"/>
+<contactref element="U$3" pad="GND"/>
+<contactref element="U$3" pad="GND#2"/>
+<wire x1="64.77" y1="71.08" x2="59.429528125" y2="75.723040625" width="0" layer="19" extent="1-1"/>
+<wire x1="48.26" y1="67.31" x2="59.429528125" y2="75.723040625" width="0" layer="19" extent="1-1"/>
+<wire x1="45.72" y1="51.93" x2="48.26" y2="67.31" width="0" layer="19" extent="1-1"/>
+<wire x1="52.07" y1="44.58" x2="45.72" y2="51.93" width="0" layer="19" extent="1-1"/>
+<wire x1="57.15" y1="44.58" x2="52.07" y2="44.58" width="0" layer="19" extent="1-1"/>
+<wire x1="62.23" y1="44.45" x2="57.15" y2="44.58" width="0" layer="19" extent="1-1"/>
+<wire x1="63.5" y1="50.8" x2="62.23" y2="44.45" width="0" layer="19" extent="1-1"/>
 </signal>
 <signal name="VCC">
 <contactref element="U$1" pad="VCC"/>
+<contactref element="IC2" pad="2"/>
+<contactref element="C2" pad="1"/>
+<contactref element="U$2" pad="VCC"/>
+<wire x1="59.47294375" y1="72.98791875" x2="67.05" y2="63.78" width="0" layer="19" extent="1-1"/>
+<wire x1="66.04" y1="50.8" x2="67.05" y2="63.78" width="0" layer="19" extent="1-1"/>
+<wire x1="57.15" y1="41.78" x2="66.04" y2="50.8" width="0" layer="19" extent="1-1"/>
 </signal>
 <signal name="N$2">
-<contactref element="IC2" pad="3"/>
+<contactref element="JP1" pad="2"/>
 <contactref element="U$4" pad="C"/>
-<wire x1="22.86" y1="29.21" x2="64.77" y2="71.08" width="0" layer="19" extent="1-1"/>
+<wire x1="22.86" y1="29.21" x2="62.23" y2="46.99" width="0" layer="19" extent="1-1"/>
 </signal>
 </signals>
